File: electronica/eagle/Shield_arduinoYUN/shield_digitales.brd (EAGLE design)
At the start: 100 x 80 mm, 10 parts, among them Q1 IRF540, U1 YUN_MINI_SHIELD-BPLACE

Commit message: placa
Parts:
- moved TEMPERATURA 20.8 mm to (45.7, 26.0), turned to 180 degrees
- moved HUMEDAD 7.85 mm to (27.3, 45.7)
- moved SONAR 5.12 mm to (64.1, 31.8), turned to 270 degrees
- moved R2 4.26 mm to (59.1, 39.4), turned to 180 degrees
- moved R3 3.81 mm to (27.3, 27.9)
- moved FOTORESIS 2.54 mm to (34.9, 35.6)
Connections:
- removed net 12V: MOTOR.1
- net DATA: now also U1.D2; no longer U1.D5
- net ECHO: now also U1.D4; no longer U1.D3
- net GND: now also MOTOR.1
- net PWM: now also U1.D5; no longer U1.D6
- net TRIG: now also U1.D3; no longer U1.D4
Routing:
- net DATA: track 6.88 -> 28.7 mm
- net ANALOG: track 3.81 -> 12.6 mm
- net ECHO: track 9.94 -> 5.71 mm
- net TRIG: track 9.20 -> 5.71 mm
- net PWM: track 6.50 -> 9.42 mm
- net FOTORESISTENCIA: track 15.9 -> 13.3 mm
- net 5V: track 61.7 -> 59.6 mm
- net N$1: track 9.42 -> 10.7 mm
